File: Backups/SD Card Version/Jarvis.sch (KiCad schematic (older format))
At the start: 124 parts, among them IC1 ADP1607, IC2 MAX-8Q, IC3 MPU-9250, IC4 STM32F411CxUx, IC5 Si4460, IC6 MS5611-01BA03, IC7 S25FL127S, J1 PYRO, J2 PWR, J3 ARM, J4 MICROUSB, P1 SMA, P2 SMA, P3 SWD_TC, Q1 PFET, Q2 PFET, Q3 PFET, Q4 NFET, Q5 NFET, Q6 NFET, Q7 NFET, X1 434MHz ANT, X10 Housing x1, X11 Housing x3, X12 M Crimps x6, X13 F Crimps x17, X14 Crimp Tool, X2 Red LED, X3 AA Battery, X4 AA Holder, X5 ARM Switch, X6 Wire, X7 Heat Shrink, X8 Housing x1, X9 Housing x4, Y1 26MHz, Y2 30MHz

Commit message: Replaced SD Card with 16MB Flash and started placment
Parts:
- removed IC7: S25FL127S, agg:WND008, symbol S25FL127S
- removed J4: MICROUSB, agg:MICROUSB_MOLEX_47589-0001, symbol MICROUSB
- added C29: 100nF, agg:0402-L, symbol C_Small
- added R27, R28, R29, R30, R31: 47K, agg:0402-L, symbol R
- added TP1, TP10, TP11, TP12, TP13, TP14, TP15, TP16, TP17, TP18, TP19, TP2, TP20, TP3, TP4, TP5, TP6, TP7, TP8, TP9: TESTPAD, agg:TESTPAD, symbol TESTPAD
- added U1: MICROSD, agg:MICROSD_MOLEX_503398-1892, symbol MICROSD
Connections:
- net labels added: SDIO_CK, SDIO_CMD, SDIO_D0, SDIO_D1, SDIO_D2, SDIO_D3, SD_CD, SPI4_MISO, SPI4_MOSI, SPI4_NSS1, SPI4_SCK, SPI5_MISO, SPI5_MOSI, SPI5_NSS1, SPI5_SCK, USART2_RX, USART2_TX, nIRQ
- net labels removed: Radio_nIRQ, SPI1_MISO, SPI1_MOSI, SPI1_NSS1_FLASH, SPI1_NSS2_RADIO, SPI1_SCK, SPI2_MISO, SPI2_MOSI, SPI2_NSS1_MPU, SPI2_SCK, USART1_RX, USART1_TX, USB_OTG_DM, USB_OTG_DP
- wire segments 311 -> 448
- no-connect marks 25 -> 16
Other:
- note added: "TODO: Add Test Points & M2 Mounts"
- note removed: "TODO: Add Test Points"
- moved on the sheet: D10, D5, D6, J2, J3
