File: Ground Station/Ground Station.kicad_pcb (KiCad board)
At the start: 4 copper layers, 44 x 16 mm, 55 parts, among them IC1 ADP3335, IC2 STM32F042F6P6, IC3 Si4460, IC4 S25FL127S, J1 USB-PLUG, P1 SMA, P2 SWD_TC, X1 RF Frame, Y1 30MHz, Y2 26MHz

Commit message: Corrected Radio Passives in Ground Station
Parts:
- C1: value 5.1pF -> 3pF
- C3: value 2.7pF -> 1.2pF
- C4: value 18pF -> 33pF
- C7, C9: value 8.2pF -> 5.1pF
- C8: value 15pF -> 10pF
- L1: value 56nH -> 18nH
- L2: value 56nH -> 22nH
- L3, L4: value 18nH -> 6.8nH
- L5: value 56nH -> 8.2nH
- L6: value 220nH -> 120nH
Changed lines of the file:
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@@
-(kicad_pcb (version 4) (host pcbnew 4.0.2-4+6225~38~ubuntu14.04.1-stable)
+(kicad_pcb (version 4) (host pcbnew 4.0.2+e4-6225~38~ubuntu14.04.1-stable)
   (general
-    (links 126)
-    (no_connects 0)
-    (area 122.472599 92.4726 180.3274 117.1774)
+    (links 131)
+    (no_connects 4)
+    (area 131.949999 93.949999 176.050001 110.050001)
     (thickness 1.6)
     (drawings 48)
@@
       (effects (font (size 1 1) (thickness 0.15)))
     )
-    (fp_text value 5.1pF (at 1.61 0 360) (layer F.Fab)
+    (fp_text value 3pF (at 1.61 0 360) (layer F.Fab)
       (effects (font (size 1 1) (thickness 0.15)))
     )
@@
       (effects (font (size 1 1) (thickness 0.15)))
     )
-    (fp_text value 2.7pF (at 1.61 0 270) (layer F.Fab)
+    (fp_text value 1.2pF (at 1.61 0 270) (layer F.Fab)
       (effects (font (size 1 1) (thickness 0.15)))
     )
@@
       (effects (font (size 1 1) (thickness 0.15)))
     )
-    (fp_text value 18pF (at 1.61 0 270) (layer F.Fab)
+    (fp_text value 33pF (at 1.61 0 270) (layer F.Fab)
       (effects (font (size 1 1) (thickness 0.15)))
     )
@@
       (effects (font (size 1 1) (thickness 0.15)))
     )
-    (fp_text value 8.2pF (at 1.61 0 360) (layer F.Fab)
+    (fp_text value 5.1pF (at 1.61 0 360) (layer F.Fab)
       (effects (font (size 1 1) (thickness 0.15)))
     )
@@
       (effects (font (size 1 1) (thickness 0.15)))
     )
-    (fp_text value 15pF (at 1.61 0 180) (layer F.Fab)
+    (fp_text value 10pF (at 1.61 0 180) (layer F.Fab)
       (effects (font (size 1 1) (thickness 0.15)))
     )
@@
       (effects (font (size 1 1) (thickness 0.15)))
     )
-    (fp_text value 8.2pF (at 1.61 0 180) (layer F.Fab)
+    (fp_text value 5.1pF (at 1.61 0 180) (layer F.Fab)
       (effects (font (size 1 1) (thickness 0.15)))
     )
@@
       (effects (font (size 1 1) (thickness 0.15)))
     )
-    (fp_text value 56nH (at 1.61 0 180) (layer F.Fab)
+    (fp_text value 18nH (at 1.61 0 180) (layer F.Fab)
       (effects (font (size 1 1) (thickness 0.15)))
     )
@@
       (effects (font (size 1 1) (thickness 0.15)))
     )
-    (fp_text value 56nH (at 1.61 0 270) (layer F.Fab)
+    (fp_text value 22nH (at 1.61 0 270) (layer F.Fab)
       (effects (font (size 1 1) (thickness 0.15)))
     )
@@
       (effects (font (size 1 1) (thickness 0.15)))
     )
-    (fp_text value 18nH (at 3.165 1.166428 180) (layer F.Fab)
+    (fp_text value 6.8nH (at 3.165 1.166428 180) (layer F.Fab)
       (effects (font (size 1 1) (thickness 0.15)))
     )
@@
       (effects (font (size 1 1) (thickness 0.15)))
     )
-    (fp_text value 18nH (at 1.61 0 270) (layer F.Fab)
+    (fp_text value 6.8nH (at 1.61 0 270) (layer F.Fab)
       (effects (font (size 1 1) (thickness 0.15)))
     )
@@
       (effects (font (size 1 1) (thickness 0.15)))
     )
-    (fp_text value 56nH (at 1.61 0 270) (layer F.Fab)
+    (fp_text value 8.2nH (at 1.61 0 270) (layer F.Fab)
       (effects (font (size 1 1) (thickness 0.15)))
     )
@@
       (effects (font (size 1 1) (thickness 0.15)))
     )
-    (fp_text value 220nH (at 2.025 0 360) (layer F.Fab)
-      (effects (font (size 1 1) (thickness 0.15)))
-    )
+    (fp_text value 120nH (at 2.025 0 360) (layer F.Fab)
+      (effects (font (size 1 1) (thickness 0.15)))
+    )
