File: Jarvis/Jarvis.sch (KiCad schematic (older format))
At the start: 183 parts, among them IC1 ADP1607, IC2 MAX-8Q, IC3 MPU-9250, IC4 STM32F411CxUx, IC5 Si4460, IC6 MS5611-01BA03, IC7 S25FL127S, J1 PYRO, J2 PWR, J3 ARM, J4 MICROUSB, P1 SMA, P2 SMA, P3 SWD_TC, Q1 PFET, Q2 PFET, Q3 PFET, Q4 NFET, Q5 NFET, Q6 NFET, Q7 NFET, X1 434MHz ANT, X10 Housing x1, X11 Housing x3, X12 M Crimps x6, X13 F Crimps x17, X14 Crimp Tool, X15 RF Frame, X16 RF Cover, X17 Heat Shrink, X18 Heat Shrink, X19 Heat Shrink, X2 Red LED, X3 AA Battery, X4 AA Holder, X5 ARM Switch, X6 Wire, X7 Heat Shrink, X8 Housing x1, X9 Housing x4, Y1 26MHz, Y2 30MHz

Commit message: started barometer driver
Parts:
- D1, D2, D3, D4: symbol LED -> LED-RESCUE-Jarvis
- J4: symbol MICROUSB -> MICROUSB-RESCUE-Jarvis
- P3: symbol SWD_TC -> SWD_TC-RESCUE-Jarvis
Other:
- note removed: "X1"
- note removed: "X10"
- note removed: "X11"
- note removed: "X12"
- note removed: "X13"
- note removed: "X14"
- note removed: "X2"
- note removed: "X3\n"
- note removed: "X4"
- note removed: "X5"
- note removed: "X6"
- note removed: "X7"
- note removed: "X8"
- note removed: "X9"
Changed lines of the file:
@@
-EESchema Schematic File Version 2
+EESchema Schematic File Version 3
+LIBS:Jarvis-rescue
 LIBS:power
 LIBS:device
-LIBS:transistors
-LIBS:conn
 LIBS:linear
 LIBS:regul
-LIBS:74xx
-LIBS:cmos4000
 LIBS:adc-dac
 LIBS:memory
@@
 LIBS:digital-audio
 LIBS:philips
-LIBS:display
 LIBS:cypress
 LIBS:siliconi
@@
 LIBS:atmel
 LIBS:contrib
-LIBS:valves
+LIBS:agg-kicad
+LIBS:sma
 LIBS:Jarvis-cache
-EELAYER 25 0
+EELAYER 26 0
 EELAYER END
 $Descr A3 16535 11693
@@
 $EndDescr
 $Comp
-L SWD_TC P3
+L SWD_TC-RESCUE-Jarvis P3
 U 1 1 56EB1724
 P 2600 7600
@@
 $EndComp
 $Comp
-L LED D1
+L LED-RESCUE-Jarvis D1
 U 1 1 56F5ECA6
 P 12650 4800
@@
 $EndComp
 $Comp
-L LED D4
+L LED-RESCUE-Jarvis D4
 U 1 1 56F61B35
 P 15000 4800
@@
 COMPLETE
 $Comp
-L LED D2
+L LED-RESCUE-Jarvis D2
 U 1 1 56FE9FC1
 P 13450 4800
@@
 $EndComp
 $Comp
-L LED D3
+L LED-RESCUE-Jarvis D3
 U 1 1 56FEA13F
 P 14200 4800
@@
 Text Notes 8450 9700 0    47   ~ 0
 External HBT & Status\nindication will be done\nthrough sounder & radio
-Text Notes 4448 9197 0    47   ~ 9
-X2
-Text Notes 4448 9268 0    47   ~ 9
-X3\n
-Text Notes 4448 9339 0    47   ~ 9
-X4
-Text Notes 4448 9409 0    47   ~ 9
-X5
 $Comp
 L C_Small C28
@@
 Text Notes 8000 5750 0    60   Italic 0
 COMPLETE
-Text Notes 4451 9479 0    47   ~ 9
-X6
-Text Notes 4450 9551 0    47   ~ 9
-X7
-Text Notes 6051 9195 0    47   ~ 9
-X9
-Text Notes 6049 9267 0    47   ~ 9
-X10
-Text Notes 6050 9335 0    47   ~ 9
-X11
-Text Notes 6050 9407 0    47   ~ 9
-X12
-Text Notes 6050 9478 0    47   ~ 9
-X13
-Text Notes 6051 9549 0    47   ~ 9
-X14
 $Comp
 L GND #PWR0101
@@
 $EndComp
 $Comp
-L MICROUSB J4
+L MICROUSB-RESCUE-Jarvis J4
 U 1 1 5705CFA8
 P 12600 6500
@@
 Text Notes 8450 9050 0    55   ~ 11
 Notes:
-Text Notes 7000 9250 0    47   ~ 0
+Text Notes 7150 9250 0    47   ~ 0
 X17 Red Heatshrink\nX18 Blue Heatshrink\nX19 Yellow Heatshrink
-Text Notes 6050 9123 0    47   ~ 9
-X8
 Text Notes 6050 9550 0    47   ~ 0
 X8 3 Pin Housing\nX9 2 Pin Housing\nX10 6 Pin Housing\nX11 2 Pin Recepticle\nX12 Male Crimps\nX13 Femal Crimps\nX14 Crimp Tool
-Text Notes 4451 9122 0    47   ~ 9
-X1
-Text Notes 4450 9550 0    47   ~ 0
+Text Notes 4400 9550 0    47   ~ 0
 X1 434MHz Stubby Radio Antenna\nX2 Red Indicator LED for Pyro Arming\nX3 Energizer L91 Lithium Ultimate AA\nX4 AA Battery Holder\nX5 Key Switch for Arming Pyrotechnics\nX6 Wire\nX7 Black Heatshrink
 Text Notes 8450 9220 0    47   ~ 0
